Commit message: 空地协同出击

File: workspace/swarm_defense_ws/src/car3_control/urdf/car3.xacro (robot description, xacro)
@@ -30,5 +30,5 @@
       <origin xyz="0 0 0" rpy="0 0 0" />
       <geometry>
-        <mesh filename="package://car3/meshes/base_link.STL" />
+        <mesh filename="package://car3_control/meshes/base_link.STL" />
       </geometry>
       <material name="">
@@ -39,5 +39,5 @@
       <origin xyz="0 0 0.004" rpy="0 0 0" />
       <geometry>
-        <mesh filename="package://car3/meshes/base_link.STL" />
+        <mesh filename="package://car3_control/meshes/base_link.STL" />
       </geometry>
     </collision>
@@ -53,5 +53,5 @@
       <origin xyz="0 0 0" rpy="0 0 0" />
       <geometry>
-        <mesh filename="package://car3/meshes/wheel_lf_link.STL" />
+        <mesh filename="package://car3_control/meshes/wheel_lf_link.STL" />
       </geometry>
       <material name="">
@@ -93,5 +93,5 @@
       <origin xyz="0 0 0" rpy="0 0 0" />
       <geometry>
-        <mesh filename="package://car3/meshes/wheel_rf_link.STL" />
+        <mesh filename="package://car3_control/meshes/wheel_rf_link.STL" />
       </geometry>
       <material name="">
@@ -133,5 +133,5 @@
       <origin xyz="0 0 0" rpy="0 0 0" />
       <geometry>
-        <mesh filename="package://car3/meshes/wheel_lb_link.STL" />
+        <mesh filename="package://car3_control/meshes/wheel_lb_link.STL" />
       </geometry>
       <material name="">
@@ -173,5 +173,5 @@
       <origin xyz="0 0 0" rpy="0 0 0" />
       <geometry>
-        <mesh filename="package://car3/meshes/wheel_rb_link.STL" />
+        <mesh filename="package://car3_control/meshes/wheel_rb_link.STL" />
       </geometry>
       <material name="">
@@ -212,5 +212,5 @@
       <origin xyz="0 0 0" rpy="0 0 0" />
       <geometry>
-        <mesh filename="package://car3/meshes/laser_link.STL" />
+        <mesh filename="package://car3_control/meshes/laser_link.STL" />
       </geometry>
       <material name="">
@@ -221,5 +221,5 @@
       <origin xyz="0 0 0" rpy="0 0 0" />
       <geometry>
-        <mesh filename="package://car3/meshes/laser_link.STL" />
+        <mesh filename="package://car3_control/meshes/laser_link.STL" />
       </geometry>
     </collision>
@@ -240,5 +240,5 @@
       <origin xyz="0 0 0" rpy="0 0 0" />
       <geometry>
-        <mesh filename="package://car3/meshes/imu_link.STL" />
+        <mesh filename="package://car3_control/meshes/imu_link.STL" />
       </geometry>
       <material name="">
@@ -249,5 +249,5 @@
       <origin xyz="0 0 0" rpy="0 0 0" />
       <geometry>
-        <mesh filename="package://car3/meshes/imu_link.STL" />
+        <mesh filename="package://car3_control/meshes/imu_link.STL" />
       </geometry>
     </collision>
