Commit message: 空地协同：新增 V型封控围捕包与入侵视角采集，入侵小车(car2)带红色物块
- 新增 air_vblock_capture 独立包（V型封控围捕，不影响 Voronoi 方案）
- 新增 intruder_car_capture / intruder_view_capture 视角采集（代码，不含图片数据）
- 新增 gimbal_camera 云台相机部件与演示脚本
- 新增 run_vblock_capture_*.sh 一键脚本、V型封控定稿/调参/可调参数清单文档
- car3.xacro 新增 red_marker 参数：外墙左上角入侵小车(car2)加红色入侵物块（仅视觉）
- air_intruder_pursuit 支持 CORNER_2 出生，紧阵型偏移参数化（encircle_*）
- 同步 launch_air_intruder_sim.sh 的 UAV 速度/加速度参数与 nesting_room 世界/模型更新

Co-Authored-By: Claude Opus 4.7 <noreply@anthropic.com>

File: workspace/swarm_defense_ws/src/car3_control/urdf/car3.xacro (robot description, xacro)
@@ -6,4 +6,5 @@
   <xacro:arg name="prefix" default=""/>
   <xacro:arg name="ns" default="/"/>
+  <xacro:arg name="red_marker" default="false"/>
   <xacro:property name="pfx" value="$(arg prefix)"/>
   <xacro:property name="robot_ns" value="$(arg ns)"/>
@@ -385,3 +386,40 @@
     </sensor>
   </gazebo>
+  <!-- 入侵标识：红色物块（仅视觉，无碰撞）。尺寸/位置与 intruder_car_capture
+       的 car3_red 一致：0.08 立方体，base_link z 0.13（贯穿雷达-车身柱、贴合车身、
+       不挡雷达，顶 0.17 < 雷达底 0.2356）。默认关闭，开启后不参与任何物理/导航。 -->
+  <xacro:if value="$(arg red_marker)">
+    <link name="${pfx}intruder_marker">
+      <inertial>
+        <mass value="0.0001" />
+        <origin xyz="0 0 0" rpy="0 0 0"/>
+        <inertia ixx="1e-8" ixy="0" ixz="0" iyy="1e-8" iyz="0" izz="1e-8" />
+      </inertial>
+      <visual>
+        <origin xyz="0 0 0" rpy="0 0 0" />
+        <geometry>
+          <box size="0.08 0.08 0.08" />
+        </geometry>
+        <material name="intruder_red">
+          <color rgba="1 0 0 1" />
+        </material>
+      </visual>
+    </link>
+    <joint name="${pfx}intruder_marker_joint" type="fixed">
+      <origin xyz="0 0 0.13" rpy="0 0 0" />
+      <parent link="${pfx}base_link" />
+      <child link="${pfx}intruder_marker" />
+    </joint>
+    <gazebo reference="${pfx}intruder_marker">
+      <material>Gazebo/Red</material>
+      <visual>
+        <material>
+          <ambient>1 0 0 1</ambient>
+          <diffuse>1 0 0 1</diffuse>
+          <specular>0.5 0 0 1</specular>
+          <emissive>0.4 0 0 1</emissive>
+        </material>
+      </visual>
+    </gazebo>
+  </xacro:if>
 </robot>

Commit message: SWARM-LIO 空地同场(M6)定稿:car0/car1 地面车接入 SWARM-LIO 定位 + gazebo 真值世界对齐 + 各自 2D 导航
两辆围捕小车与 UAV 共用一个对齐世界(quad0/world),各车独立 SWARM-LIO 定位并完成 2D 导航。

- 新增 car3_lio/:run_m6_air_ground_demo.sh(M6 分段一键演示 clean/up_world/up_uavlio/up_carlio/up_scan/up_align/up_nav/up_takeoff/verify/status)、run_m3_align_demo.sh、car0/car1_sim.yaml、env.sh、m3_verify.py、mapping_drive.py、patch_guard_launch.py 与完成说明文档
- car3_control:urdf/car3.xacro 增 lidar=mid360_lio 平装分支;新增 car0_nav.launch/car1_nav.launch(car1 整栈包 group ns=car1,与 car0 根命名空间同场并存)、params_car0/params_car1、maps/car0_nav_map、mid360_to_scan/build_lio_2d_map/build_scan_2d_map.py
- car3_swarm:car_spawn.launch 参数化 lidar;新增 lio_car_bringup/dual_lio_car_bringup 车端 launch、map_alignment.py(gazebo 真值世界对齐)、lio_pose_guard.py、uav_offboard_takeoff_lio_ref.py、ego_lio_to_px4_bridge.py、lio_cloud_to_px4.cpp
- 新增根文档 空地协同围捕项目框架.md

Co-Authored-By: Claude Opus 4.7 <noreply@anthropic.com>

File: workspace/swarm_defense_ws/src/car3_control/urdf/car3.xacro (robot description, xacro)
@@ -7,5 +7,13 @@
   <xacro:arg name="ns" default="/"/>
   <xacro:arg name="red_marker" default="false"/>
+  <!-- lidar: hokuyo(2D, 默认) / mid360(3D PointCloud2, 旧 mid360_car3 用) /
+       mid360_lio(3D CustomMsg 平装, 与 UAV 同款 liblivox_laser_simulation.so, 供 SWARM-LIO) -->
+  <xacro:arg name="lidar" default="hokuyo"/>
+  <xacro:arg name="livox_samples" default="24000"/>
+  <!-- mid360_lio 专用: lidar/imu 绝对话题名(不受 robotNamespace 影响), 默认单机用 /car0 -->
+  <xacro:arg name="lio_lidar_topic" default="/car0/livox/lidar"/>
   <xacro:property name="pfx" value="$(arg prefix)"/>
+  <xacro:property name="lidar_type" value="$(arg lidar)"/>
+  <xacro:property name="livox_samples_val" value="$(arg livox_samples)"/>
   <xacro:property name="robot_ns" value="$(arg ns)"/>
   <link name="${pfx}base_footprint">
@@ -204,4 +212,5 @@
     </actuator>
   </transmission>
+  <xacro:if value="${lidar_type == 'hokuyo'}">
   <link name="${pfx}laser_link">
     <inertial>
@@ -231,4 +240,35 @@
     <child link="${pfx}laser_link" />
   </joint>
+  </xacro:if>
+  <!-- lidar=mid360/mid360_lio: 3D 雷达替换 2D hokuyo（外观 mesh + livox 点云），传感器原点即 livox_link。
+       livox_link 平装(rpy 0)于 base_link 上方 z=0.24, device z 轴竖直; 不斜装。 -->
+  <xacro:if value="${lidar_type == 'mid360' or lidar_type == 'mid360_lio'}">
+  <link name="${pfx}livox_link">
+    <inertial>
+      <mass value="0.265" />
+      <inertia ixx="0.00002" ixy="0" ixz="0" iyy="0.00002" iyz="0" izz="0.00001" />
+    </inertial>
+    <visual>
+      <origin xyz="0 0 0" rpy="0 0 0" />
+      <geometry>
+        <mesh filename="package://livox_laser_simulation/meshes/mid360.dae" />
+      </geometry>
+      <material name="">
+        <color rgba="0.2 0.2 0.2 1" />
+      </material>
+    </visual>
+    <collision>
+      <origin xyz="0 0 0" rpy="0 0 0" />
+      <geometry>
+        <mesh filename="package://livox_laser_simulation/meshes/mid360_rules.dae" />
+      </geometry>
+    </collision>
+  </link>
+  <joint name="livox_joint" type="fixed">
+    <origin xyz="0 0 0.24" rpy="0 0 0" />
+    <parent link="${pfx}base_link" />
+    <child link="${pfx}livox_link" />
+  </joint>
+  </xacro:if>
   <link name="${pfx}imu_link">
     <inertial>
@@ -334,4 +374,5 @@
     </plugin>
   </gazebo>
+  <xacro:if value="${lidar_type == 'hokuyo'}">
   <gazebo reference="${pfx}laser_link">
     <material>Gazebo/Black</material>
@@ -366,4 +407,102 @@
     </sensor>
   </gazebo>
+  </xacro:if>
+  <!-- lidar=mid360: livox 仿真插件 ray sensor，按 mid360.csv 逐点扫描发 PointCloud2 -->
+  <xacro:if value="${lidar_type == 'mid360'}">
+  <gazebo reference="${pfx}livox_link">
+    <material>Gazebo/Black</material>
+    <sensor type="ray" name="${pfx}livox_link">
+      <pose>0 0 0 0 0 0</pose>
+      <visualize>false</visualize>
+      <update_rate>10</update_rate>
+      <always_on>true</always_on>
+      <plugin name="gazebo_ros_livox_controller" filename="liblivox_laser_simulation.so">
+        <ray>
+          <scan>
+            <horizontal>
+              <samples>100</samples>
+              <resolution>1</resolution>
+              <min_angle>0</min_angle>
+              <max_angle>6.28319</max_angle>
+            </horizontal>
+            <vertical>
+              <samples>360</samples>
+              <resolution>1</resolution>
+              <min_angle>-0.0562</min_angle>
+              <max_angle>0.9812</max_angle>
+            </vertical>
+          </scan>
+          <range>
+            <min>0.1</min>
+            <max>30</max>
+            <resolution>0.02</resolution>
+          </range>
+          <noise>
+            <type>gaussian</type>
+            <mean>0.0</mean>
+            <stddev>0.0</stddev>
+          </noise>
+        </ray>
+        <visualize>false</visualize>
+        <samples>${livox_samples_val}</samples>
+        <downsample>1</downsample>
+        <csv_file_name>package://livox_laser_simulation/scan_mode/mid360.csv</csv_file_name>
+        <ros_topic>scan</ros_topic>
+      </plugin>
+    </sensor>
+  </gazebo>
+  </xacro:if>
+  <!-- lidar=mid360_lio: SWARM-LIO 专用。与 UAV 的 iris_mid360_N 完全同款的 CustomMsg 插件
+       (liblivox_laser_simulation.so + publish_pointcloud_type=3 = livox_ros_driver2/CustomMsg)。
+       livox_link 与 mid360 分支共用(平装 rpy 0)。csv 由插件经 model://Mid360/scan_mode/ 解析,
+       故 GAZEBO_MODEL_PATH 需含 livox 包 models。话题用 lio_lidar_topic 绝对名。 -->
+  <xacro:if value="${lidar_type == 'mid360_lio'}">
+  <gazebo reference="${pfx}livox_link">
+    <material>Gazebo/Black</material>
+    <sensor type="ray" name="${pfx}livox_lio_sensor">
+      <pose>0 0 0 0 0 0</pose>
+      <visualize>false</visualize>
+      <always_on>true</always_on>
+      <update_rate>10</update_rate>
+      <plugin name="${pfx}gazebo_livox_lio_controller" filename="liblivox_laser_simulation.so">
+        <ray>
+          <scan>
+            <horizontal>
+              <samples>100</samples>
+              <resolution>1</resolution>
+              <min_angle>-1.57</min_angle>
+              <max_angle>1.57</max_angle>
+            </horizontal>
+            <vertical>
+              <samples>360</samples>
+              <resolution>1</resolution>
+              <min_angle>-1.57</min_angle>
+              <max_angle>1.57</max_angle>
+            </vertical>
+          </scan>
+          <range>
+            <min>0.1</min>
+            <max>45</max>
+            <resolution>0.02</resolution>
+          </range>
+          <noise>
+            <type>gaussian</type>
+            <mean>0.0</mean>
+            <stddev>0.0</stddev>
+          </noise>
+        </ray>
+        <publish_scan_visualization>false</publish_scan_visualization>
+        <samples>18000</samples>
+        <downsample>2</downsample>
+        <csv_file_name>mid360-real-centr.csv</csv_file_name>
+        <publish_pointcloud_type>3</publish_pointcloud_type>
+        <ros_topic>$(arg lio_lidar_topic)</ros_topic>
+        <frameName>${pfx}livox_link</frameName>
+        <enable_self_filter>false</enable_self_filter>
+        <debug>false</debug>
+      </plugin>
+    </sensor>
+  </gazebo>
+  </xacro:if>
   <gazebo reference="${pfx}imu_link">
     <material>Gazebo/Orange</material>
@@ -375,4 +514,5 @@
       <topic>__default_topic__</topic>
       <plugin filename="libgazebo_ros_imu_sensor.so" name="imu_plugin">
+        <robotNamespace>${robot_ns}</robotNamespace>
         <topicName>imu</topicName>
         <bodyName>${pfx}imu_link</bodyName>
